File: hardware/Для изготовления/Печатная плата/Печатная плата принимающая ось X/Печатная плата принимающая ось X.brd (EAGLE design)
At the start: 60.4 x 38.1 mm, 10 parts, among them J1 22-03-5035

Commit message: принимающие платы разделены по осям
Other:
- board size 60.4 x 38.1 mm -> 30.4 x 68.1 mm
Changed lines of the file:
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@@
 <setting verticaltext="up"/>
 </settings>
-<grid distance="10" unitdist="mm" unit="mm" style="lines" multiple="1" display="no" altdistance="5" altunitdist="mm" altunit="mm"/>
+<grid distance="10" unitdist="mm" unit="mm" style="lines" multiple="1" display="no" altdistance="5" altunitdist="mil" altunit="mm"/>
 <layers>
 <layer number="1" name="Top" color="4" fill="1" visible="yes" active="yes"/>
@@
 <board>
 <plain>
-<wire x1="-13.871" y1="-1.143" x2="46.533" y2="-1.143" width="0" layer="20"/>
-<wire x1="46.533" y1="-1.143" x2="46.533" y2="36.947" width="0" layer="20"/>
-<wire x1="46.533" y1="36.947" x2="-13.871" y2="36.947" width="0" layer="20"/>
-<wire x1="-13.871" y1="36.947" x2="-13.871" y2="-1.143" width="0" layer="20"/>
+<wire x1="16.129" y1="-1.143" x2="46.533" y2="-1.143" width="0" layer="20"/>
+<wire x1="46.533" y1="-1.143" x2="46.533" y2="66.947" width="0" layer="20"/>
+<wire x1="46.533" y1="66.947" x2="16.129" y2="66.947" width="0" layer="20"/>
+<wire x1="16.129" y1="66.947" x2="16.129" y2="-1.143" width="0" layer="20"/>
 <hole x="17.907" y="34.925" drill="3"/>
 <hole x="17.907" y="0.762" drill="3"/>
 <hole x="44.577" y="0.762" drill="3"/>
 <hole x="44.704" y="35.052" drill="3"/>
-<hole x="0" y="30" drill="8.2"/>
-<hole x="0" y="5" drill="8.2"/>
+<hole x="31.496" y="53.848" drill="8.2"/>
 </plain>
 <attributes>
