File: hardware/Для изготовления/Печатная плата/Печатная плата принимающая ось X/Печатная плата принимающая ось X.sch (EAGLE design)
At the start: 23 parts, among them J1 POWER_JACK, Q1 IRF540

Commit message: принимающие платы разделены по осям
Parts:
- removed J10, J4, J5, J6, J7, J8, J9: (no value), Wurth_Elektronik_Electromechanic_Input-Output_Connectors_rev16a:615006138421
- removed J11, J12, J3: (no value), SparkFun-Connectors:BANANA_CONN
- removed Q1: IRF540, transistor-power:IRF540
- removed R5, R6: 330, resistor:R-EU_0204/7
- removed S1: reset_button, SparkFun-Switches:MOMENTARY-SWITCH-SPST-PTH-6.0MM
- removed U$3: WIRELESS-BLUETOOTH-HC-05, diy-modules:WIRELESS-BLUETOOTH-HC-05
- added D2: (no value), SparkFun-LED:LED5MM
- added R2: 10K, resistor:R-EU_0204/7
- J1: value POWER_JACK -> 22-03-5035; device SparkFun-Connectors:POWER_JACK -> molex:22-03-5035
- J2: device SparkFun-Connectors:BANANA_CONN -> Wurth_Elektronik_Electromechanic_Input-Output_Connectors_rev16a:615006138421
- R1: value 330 -> 10K
- R3, R4: value 330 -> (none)
- U$1: value OPENCM9.04 -> OPTICAL_ENCODER_FC-01; device OpenCM9.04:OPENCM9.04 -> other components:OPTICAL_ENCODER_FC-01
- U$2: value 5MMRGBLED -> ENDSTOP; device led_rgb:5MMRGBLED -> other components:ENDSTOP
Connections:
- removed net 5V: R6.1, U$1.5V, U$1.5V2
- removed net BLUE: R5.1, U$1.16
- removed net ENCODER_X_1: J4.6, U$1.21
- removed net ENCODER_X_2: J5.6, U$1.23
- removed net ENCODER_Y: J6.6, U$1.25
- removed net ENCODER_Z_1: J7.6, U$1.0
- removed net ENCODER_Z_2: J8.6, U$1.2
- removed net ENCODER_Z_3: J10.6, U$1.6
- removed net ENCODER_Z_4: J9.6, U$1.8
- removed net ENDSTOP_X_1: J4.5, U$1.20
- removed net ENDSTOP_X_2: J5.5, U$1.22
- removed net ENDSTOP_Y: J6.5, U$1.24
- removed net ENDSTOP_Z_1: J7.5, U$1.1
- removed net ENDSTOP_Z_2: J8.5, U$1.3
- removed net ENDSTOP_Z_3: J10.5, U$1.7
- removed net ENDSTOP_Z_4: J9.5, U$1.9
- removed net GREEN: R4.1, U$1.17
- removed net N$3: Q1.G, R1.1
- removed net N$4: R5.2, U$2.BLUE
- removed net N$5: R3.2, U$2.RED
- removed net N$6: D1.A, R6.2
- removed net N$7: J1.PWR, J2.1
- removed net PUMP: R1.2, U$1.19
- removed net RED: R3.1, U$1.18
- removed net RST: S1.2, U$1.RST
- removed net RX2: U$1.5, U$3.TX
- removed net TX2: U$1.4, U$3.RX
- new net ENCODER: J2.6, R2.2, R4.2, U$1.DO
- new net ENDSTOP: J2.5, R1.2, R3.1, U$2.NO
- net 12V: now also J1.VCC, J2.2; no longer J10.2, J3.1, J4.2, J5.2, J6.2, J7.2, J8.2, J9.2, Q1.S, U$1.VCC, U$1.VCC2
- net 3.3V: now also J2.3, U$1.VCC, U$2.NC; no longer J10.3, J4.3, J5.3, J6.3, J7.3, J8.3, J9.3, U$1.3.3V, U$3.+5V
- net GND: now also D2.C, J2.4, R1.1, R2.1; no longer J1.GNDBREAK, J10.4, J12.1, J4.4, J5.4, J6.4, J7.4, J8.4, J9.4, S1.1, U$1.GND2, U$1.GND3, U$2.GND, U$3.GND
- net N$1: now also D2.A, R3.2; no longer J11.1, Q1.D
- net N$2: now also D1.A, R4.1; no longer R4.2, U$2.GREEN
- net RX/TX: now also J1.RX/TX, J2.1; no longer J10.1, J4.1, J5.1, J6.1, J7.1, J8.1, J9.1, U$1.TTL
Other:
- note removed: "+12V"
- note removed: "Axis X"
- note removed: "Axis Y"
- note removed: "Axis Z"
- note removed: "Indication"
- note removed: "Main"
- note removed: "Power"
- note removed: "Power indication"
- note removed: "Wireless module"
- moved on the sheet: D1, R1, R3, R4
